File: AQ_sensor_GSM.brd (EAGLE design)
At the start: 110 x 64 mm, 49 parts, among them IC2 MCP73831/OT, J1 F-1X03-SIP-100-32, SW1 PCM12SMTR, SW2 PCM12SMTR, U2 TEXAS_INSTRUMENTS_SN74HC125TE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, U3 TEXAS_INSTRUMENTS_LM1117IMP-3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, X1 53048-08, X2 SIMLOCK-C707_10M006_512_2, X4 50 Ohms

Commit message: Added manufacturing files
Routing:
- net GND: track 71.6 -> 39.2 mm
Changed lines of the file:
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@@
 <contactref element="D1" pad="1"/>
 <contactref element="PMS" pad="C"/>
-<wire x1="31.46" y1="2.332" x2="28.368" y2="2.332" width="0.3" layer="1"/>
-<wire x1="27" y1="3.7" x2="27" y2="6" width="0.3" layer="1"/>
-<wire x1="28.368" y1="2.332" x2="27" y2="3.7" width="0.3" layer="1"/>
 <via x="38.4" y="1" extent="1-16" drill="0.35"/>
 <via x="38.4" y="2.8" extent="1-16" drill="0.35"/>
 <via x="38.4" y="4.3" extent="1-16" drill="0.35"/>
-<via x="29.9" y="1.2" extent="1-16" drill="0.35"/>
-<via x="29.8" y="3" extent="1-16" drill="0.35"/>
-<via x="29.8" y="4.5" extent="1-16" drill="0.35"/>
-<wire x1="29.8" y1="6" x2="29.8" y2="4.5" width="0.4" layer="1"/>
-<wire x1="29.8" y1="4.5" x2="29.8" y2="3" width="0.4" layer="1"/>
-<wire x1="29.8" y1="3" x2="29.8" y2="1.3" width="0.4" layer="1"/>
-<wire x1="29.8" y1="1.3" x2="29.9" y2="1.2" width="0.4" layer="1"/>
-<wire x1="29.9" y1="1.2" x2="28.3" y2="1.2" width="0.4" layer="1"/>
 <via x="28.3" y="1.2" extent="1-16" drill="0.35"/>
-<wire x1="28.3" y1="1.2" x2="28.3" y2="2.264" width="0.4" layer="1"/>
-<wire x1="28.3" y1="2.264" x2="28.368" y2="2.332" width="0.4" layer="1"/>
-<wire x1="28.368" y1="2.332" x2="28.368" y2="2.868" width="0.4" layer="1"/>
-<wire x1="28.368" y1="2.868" x2="28.4" y2="2.9" width="0.4" layer="1"/>
-<wire x1="28.4" y1="2.9" x2="28.5" y2="3" width="0.4" layer="1"/>
-<via x="28.4" y="2.9" extent="1-16" drill="0.35"/>
-<wire x1="28.4" y1="2.9" x2="28.4" y2="4.4" width="0.4" layer="1"/>
 <via x="28.4" y="4.4" extent="1-16" drill="0.35"/>
-<wire x1="28.4" y1="4.4" x2="29.7" y2="4.4" width="0.4" layer="1"/>
-<wire x1="29.7" y1="4.4" x2="29.8" y2="4.5" width="0.4" layer="1"/>
 <wire x1="35.4" y1="6" x2="35.5" y2="5.9" width="0.4" layer="1"/>
-<wire x1="35.5" y1="5.9" x2="35.5" y2="5.2" width="0.4" layer="1"/>
-<wire x1="35.5" y1="5.2" x2="35.8" y2="4.9" width="0.4" layer="1"/>
-<wire x1="37.8" y1="4.9" x2="38.4" y2="4.3" width="0.4" layer="1"/>
-<wire x1="35.8" y1="4.9" x2="37.8" y2="4.9" width="0.4" layer="1"/>
 <via x="39.9" y="1" extent="1-16" drill="0.35"/>
-<via x="39.9" y="2.7" extent="1-16" drill="0.35"/>
-<via x="39.8" y="4.3" extent="1-16" drill="0.35"/>
-<wire x1="39.8" y1="4.3" x2="39.6" y2="4.3" width="0.4" layer="1"/>
-<wire x1="39.6" y1="4.3" x2="39.3" y2="4.6" width="0.4" layer="1"/>
-<wire x1="39.3" y1="4.6" x2="38.7" y2="4.6" width="0.4" layer="1"/>
-<wire x1="38.7" y1="4.6" x2="38.4" y2="4.3" width="0.4" layer="1"/>
-<wire x1="38.4" y1="4.3" x2="38.4" y2="2.8" width="0.4" layer="1"/>
-<wire x1="38.4" y1="2.8" x2="38.4" y2="1" width="0.4" layer="1"/>
-<wire x1="38.4" y1="1" x2="39.9" y2="1" width="0.4" layer="1"/>
-<wire x1="39.9" y1="1" x2="39.9" y2="2.7" width="0.4" layer="1"/>
-<wire x1="39.9" y1="2.7" x2="39.8" y2="2.8" width="0.4" layer="1"/>
-<wire x1="39.8" y1="2.8" x2="39.8" y2="4.3" width="0.4" layer="1"/>
 <via x="76.8" y="23.7" extent="1-16" drill="0.35"/>
 <via x="79.1" y="23.7" extent="1-16" drill="0.35"/>
@@
 <via x="80.9" y="49" extent="1-16" drill="0.35"/>
 <via x="82.2" y="49" extent="1-16" drill="0.35"/>
+<via x="28.3" y="2.9" extent="1-16" drill="0.35"/>
+<via x="29.6" y="4.4" extent="1-16" drill="0.35"/>
+<via x="29.6" y="2.8" extent="1-16" drill="0.35"/>
+<via x="29.6" y="1.2" extent="1-16" drill="0.35"/>
+<via x="39.9" y="4.4" extent="1-16" drill="0.35"/>
+<via x="39.9" y="2.8" extent="1-16" drill="0.35"/>
 <wire x1="15.825" y1="8.84" x2="15.825" y2="5.03" width="0" layer="19" extent="1-1"/>
 </signal>
