File: src/AQ_sensor_GSM.sch (EAGLE design)
At the start: 45 parts, among them IC2 MCP73831/OT, J1 F-1X03-SIP-100-32, SW1 PCM12SMTR, SW2 PCM12SMTR, U2 TEXAS_INSTRUMENTS_SN74HC125TE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, U3 TEXAS_INSTRUMENTS_LM1117IMP-3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, X1 53048-08, X2 SIMLOCK-C707_10M006_512_2, X4 50 Ohms

Commit message: Resolve schematic file error
Schematic file not opening on resolving git merge conflict
Parts:
- added H1, H2, H3, H4: MOUNT-PAD-ROUND2.8, AQ_sensor_GSM:MOUNT-PAD-ROUND2.8
Connections:
- net GND: now also H1.MOUNT, H2.MOUNT, H3.MOUNT, H4.MOUNT
Other:
- note added: "LAST UPDATE: 21/5/2020"
- note added: "sensors.AFRICA MRC"
- note removed: "LAST UPDATE: 05/10/2020"
- note removed: "sensors.AFRICA GSM"
- moved on the sheet: C1, C8, J1, MICRO_USB, POWER, R14, R5, SV1, SV2, SW1, U3, X1-1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
