File: src/CAMOutputs/GerberFiles/.sch (EAGLE design)
At the start: 56 parts, among them IC2 MCP73831/OT, J1 F-1X03-SIP-100-32, SW1 PCM12SMTR, U2 TEXAS_INSTRUMENTS_SN74HC125TE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, U3 TEXAS_INSTRUMENTS_LM1117IMP-3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, U4 ESP8266-12E/ESP-12E, U5 CH340G, X1 53048-08, X2 SIMLOCK-C707_10M006_512_2, X4 50 Ohms

Commit message: Changed Lipo charging IC to TP4056. Added Power Switch to the lipo Circuitry
Parts:
- removed C2, C3: 22pF, SparkFun-Capacitors:22PF-0603-50V-5%
- removed C5: 47uF, SparkFun-Capacitors:47UF-POLAR-EIA3528-10V-10%
- removed D5: 3A/40V/500mV, SparkFun-DiscreteSemi:DIODE-SCHOTTKY-B340A
- removed GPS: PINHD-1X4, Connector:PINHD-1X4
- removed JP1: PINHD-1X10, Connector:PINHD-1X10
- removed JP2: PINHD-1X1, Connector:PINHD-1X1
- removed L1: B1047AS-470M=P3, B1047AS-470M_P3:B1047AS-470M=P3
- removed PS1: ME2108A33P, ME2108A33P:ME2108A33P
- removed R2: 47k, rcl:R-EU_R0603
- removed S2: KMR621NGLFS, AQ_sensor_GSM:KMR621NGLFS
- removed U4: ESP8266-12E/ESP-12E, ESP8266-12E_ESP-12E (1):ESP8266-12E/ESP-12E
- removed U5: CH340G, CH340G (1):CH340G
- removed Y1: (no value), SparkFun-Clocks:CRYSTALPTH-HC49US
- added H1, H2, H3, H4: MOUNT-PAD-ROUND2.8, AQ_sensor_GSM:MOUNT-PAD-ROUND2.8
- added SV1, SV2: (no value), AQ_sensor_GSM:FE15-1
- added SW2: PCM12SMTR, AQ_sensor_GSM:PCM12SMTR
Connections:
- removed net 5V_REG: C5.+, D5.C, PS1.VOUT
- removed net ADC0: JP1.9, U4.ADC
- removed net CH_CTS: U5.!CTS
- removed net CH_DCD: U5.!DCD
- removed net CH_DSR: U5.!DSR
- removed net CH_DTR: U5.!DTR
- removed net CH_RI: U5.!RI
- removed net CH_RS232: U5.RS232
- removed net CH_RTS: U5.!RTS
- removed net ESP_CSO: JP1.5, U4.CS0
- removed net ESP_MISO: JP1.7, U4.MISO
- removed net ESP_MOSI: JP1.6, U4.MOSI
- removed net ESP_SCLK: JP1.4, U4.SCLK
- removed net GPS_RX: GPS.2, U4.IO9
- removed net GPS_TX: GPS.3, U4.IO10
- removed net IO16: JP1.8, U4.IO16
- removed net N$1: D5.A, L1.2, PS1.LX
- removed net N$2: R2.1, U4.EN
- removed net RXD: JP1.3, U4.RXD, U5.TXD
- removed net TXD: JP1.2, U4.TXD, U5.RXD
- removed net X1: C2.2, U5.XI, Y1.1
- removed net X2: C3.2, U5.XO, Y1.2
- new net VIN: MICRO_USB.VUSB, SW1.2
- net +3V3: now also SV1.1; no longer R2.2, U4.VCC, U5.V3
- net +5V: now also SV2.1, SW1.1; no longer GPS.1, JP1.1, MICRO_USB.VUSB, U5.VCC
- net D+: no longer U5.UD+
- net D-: no longer U5.UD-
- net DHT_LED: now also SV1.11; no longer U4.IO2
- net DHT_OUT: now also SV1.6; no longer U4.IO13
- net ESP_RST: now also SV2.3, SW2.2; no longer S2.1, U4.RESET
- net GND: now also H1.MOUNT, H2.MOUNT, H3.MOUNT, H4.MOUNT, SV1.2, SV2.2, SW1.SHIELD, SW2.1, SW2.SHIELD; no longer C2.1, C3.1, C5.-, GPS.4, JP1.10, PS1.VSS, S2.2, U4.GND, U5.GND
- net GSM_ANT: no longer JP2.1
- net GSM_RST_O: now also SV1.5; no longer U4.IO15
- net GSM_RX_O: now also SV1.8; no longer U4.IO14
- net GSM_TX_5V: now also SV1.7; no longer U4.IO12
- net PMS_LED: now also SV1.12; no longer U4.IO0
- net PMS_RX: now also SV1.13; no longer U4.IO4
- net PMS_TX: now also SV1.14; no longer U4.IO5
- net V_LIPO: no longer L1.1
Other:
- note added: "LAST UPDATE: 21/5/2020"
- note added: "sensors.AFRICA MRC"
- note removed: "LAST UPDATE: 05/10/2020"
- note removed: "sensors.AFRICA GSM"
- moved on the sheet: C1, C8, J1, MICRO_USB, POWER, R14, R5, SW1, U3, X1-1, X1-2, X1-3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
